File: electronics/armwiz-board.sch (EAGLE design)
At the start: 94 parts, among them IC3 SN74LVC1G74DCT, J1 MICRO-SDCARD-CONNECTOR-330006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, J12 CORTEX_DEBUGSMD, Q1 DMP2035U-7, Q2 DMP2035U-7, Q3 DMN2075U-7, Q4 DMN2075U-7, Q5 DMP2035U-7, U1 STM32F10XRXT6, U2 APX809, U3 MCP73831, U4 MIC5219-3.3V, X1 FH12-12S-1S

Commit message: Routing and layout.
Parts:
- removed BAT1: (no value), SparkFun-Electromechanical:BATTERY12MM
- removed C16, C17: 0.1uF, SparkFun-Capacitors:0.1UF-25V-5%(0603)
- removed J10, J9: (no value), SparkFun-Connectors:M021X02_NO_SILK
- removed J12: CORTEX_DEBUGSMD, SparkFun-Connectors:CORTEX_DEBUGSMD
- removed J3: (no value), SparkFun-Connectors:M05PTH
- removed J7, J8: (no value), SparkFun-Connectors:M04NO_SILK_ALL_ROUND
- removed R29: 10k, SparkFun-Passives:RESISTOR-ARRAY0603-ARV
- removed R34, R35: 10K, SparkFun-Resistors:10KOHM-1/10W-1%(0603)0603
- removed SJ1: JUMPER-PAD-2-NC_BY_TRACE, SparkFun-Passives:JUMPER-PAD-2-NC_BY_TRACE
- removed Y2: (no value), SparkFun-FreqCtrl:CRYSTAL32-SMD-MELF
- added C18: 0.1uF, SparkFun-Capacitors:0.1UF-25V-5%(0603)
- added R2, R4: 10K, SparkFun-Resistors:10KOHM-1/10W-1%(0603)0603
- J2: device SparkFun-Connectors:M031X03_NO_SILK -> SparkFun-Connectors:M04PTH
Connections:
- net TRST renamed MISO3
- removed net 5V: J3.5
- removed net MOSI: X1-6.1
- removed net N$10: SJ1.2, U$2.VBAT
- removed net N$102: J8.4
- removed net N$104: J8.2
- removed net N$105: J8.1
- removed net N$108: J8.3
- removed net N$110: J10.1
- removed net N$112: J9.1
- removed net N$113: J9.2
- removed net N$114: J7.1
- removed net N$115: J7.2
- removed net N$116: J7.3
- removed net N$117: J7.4
- removed net N$15: U1PORTB_L.PB5
- removed net N$16: U1PORTB_L.PB6
- removed net N$17: U1PORTB_L.PB7
- removed net N$41: U1PORTB_H.PB8
- removed net N$42: U1PORTB_H.PB9
- removed net N$94: J10.2
- removed net RTC_BATT: BAT1.+, U1AN_POWER.VBAT
- removed net RX1: J2.1, U1PORTA_H.PA10
- removed net SCK: X1-7.1
- removed net SWO: J12.SWO/TDO, R29B.1, U1PORTB_L.PB3
- removed net TX1: J2.2, U1PORTA_H.PA9
- new net MOSI3: U1PORTB_L.PB5, X1-6.1
- new net SCK3: U1PORTB_L.PB3, X1-7.1
- net 3.3V: now also C18.2, J2.4, R4.2, U1AN_POWER.VBAT; no longer C16.2, C17.2, J12.VCC, J3.4, R29A.2, R29B.2, R29C.2, R35.2
- net GND: now also C18.1, J2.2, R2.2; no longer BAT1.-, C16.1, C17.1, J12.GND@3, J12.GND@5, J12.GNDDTCT, J2.3, J3.2, R29D.1, R34.2
- net LCD_A0: now also U1PORTB_H.PB9
- net LCD_BL: now also U1PORTB_L.PB6
- net LCD_CS: now also U1PORTB_L.PB7
- net LCD_RST: now also U1PORTB_H.PB8
- net NRST: no longer J12.NRESET
- net RTC1: no longer Y2.2
- net RTC2: no longer Y2.1
- net SWDCLK: now also J2.3, R2.1; no longer J12.SWDCLK/TCK, J3.3, R29D.2, R34.1
- net SWDIO: now also J2.1, R4.1; no longer J12.SWDIO/TMS, J3.1, R29A.1, R35.1
- net TDI: no longer J12.NC/TDI, R29C.1
- net VBAT: now also U$2.VBAT; no longer SJ1.1
Other:
- note removed: "Corted Debug (10-pin)"
- note removed: "Note: Battery = CR1220"
- note removed: "Real Time Clock"
- note removed: "USART1"
- moved on the sheet: C35, C36, R19, X1-1, X1-10, X1-11, X1-12, X1-2, X1-3, X1-4, X1-5, X1-6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

Commit message: More routing.
Parts:
- C1, C12, C2, C22, C23, C26, C27, C28, C35, C36, C4, C6, C9: device PaxInstrument-T400:SPARKFUN-CAPACITORS_CAP0603-CAP -> resistor:C-EUC0402K
- C10, C11, C13, C14, C15, C18, C3, C8: device SparkFun-Capacitors:0.1UF-25V-5%(0603) -> resistor:C-EUC0402K
- C5, C7: device SparkFun-Capacitors:33PF-50V-5%-(0603) -> resistor:C-EUC0402K
- R1, R10, R11, R12, R15, R16, R17, R18, R19, R20, R21, R22, R23, R24, R25, R3, R5, R6, R7, R8, R9: device PaxInstrument-T400:SPARKFUN-RESISTORS_RESISTOR0603-RES -> resistor:R-US_R0402
- R13, R14, R2, R28, R4: device SparkFun-Resistors:10KOHM-1/10W-1%(0603)0603 -> resistor:R-US_R0402
Other:
- moved on the sheet: C1, C10, C11, C13, C15, C18, C2, C26, C27, C3, C35, C36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

Commit message: Made some changes to schematic.
Parts:
- removed C12, C22: 10uF, resistor:C-EUC0402K
- removed C23: 1uF, resistor:C-EUC0402K
- removed C28: 0.1uF, resistor:C-EUC0402K
- removed IC3: SN74LVC1G74DCT, PaxInstrument-T400:SN74LVC1G74DCT
- removed JP1: ON, SparkFun-Passives:JUMPER-2SMD-NO
- removed Q1, Q2, Q5: DMP2035U-7, PaxInstrument-T400:MOSFET-PCHANNELSMT
- removed Q3, Q4: DMN2075U-7, PaxInstrument-T400:MOSFET-NCHANNELSMT
- removed R17: 2k, resistor:R-US_R0402
- removed R18, R21, R22, R23, R5, R6, R7: 10k, resistor:R-US_R0402
- removed R20: 18.7K, resistor:R-US_R0402
- removed R24: 34K, resistor:R-US_R0402
- removed R25: 4.7k, resistor:R-US_R0402
- removed U$2: BL-5C-CONNECTOR, charlespax:BL-5C-CONNECTOR
- removed U2: APX809, PaxInstrument-T400:APX809
- removed U3: MCP73831, SparkFun-PowerIC:MCP73831
- added BAT1: (no value), PaxInstruments-Electromechanical:BATTERY12MM
- added D3: 1N4148W, SparkFun-DiscreteSemi:DIODESOD123
- added LED1: GREEN, SparkFun-LED:LED0603
- added Y2: (no value), SparkFun-FreqCtrl:CRYSTALCRYSTAL-SMD-5X3-16MHZ
- C6: value 0.1uF -> 8pF
- C9: value 4.7uF -> 8pF
- R1: POPULATE (none) -> DNP
- R3: value 2.32k (1%) -> 360R
- Y1: value (none) -> 16MHz
Connections:
- removed net 3V3EN: JP1.2, R21.2, U4.EN
- removed net BATT_STAT: C22.1, R1.2, R17.1
- removed net N$12: Q1.G, U2.!RST
- removed net N$20: Q2.D, R20.2
- removed net N$25: IC3.!SET, Q5.G, R6.2, S6.1
- removed net N$26: Q2.G, Q3.D, R5.2
- removed net N$27: IC3.!CLR, Q4.D, R7.2
- removed net N$28: IC3.Q, R21.1
- removed net PWR_ONOFF: Q4.G, R22.1
- removed net SW_PWR: Q5.D, R18.1
- removed net VBAT: C9.1, Q1.D, Q2.S, R5.1, U$2.VBAT, U3.VBAT
- removed net VBAT_EN: Q3.G, R23.2
- removed net VBAT_SENSE: C23.1, R20.1, R24.1
- new net RTC_BAT: BAT1.+, U1AN_POWER.VBAT
- net 3.3V: now also D3.A, LED1.A, S6.2; no longer Q5.S, R1.1, U1AN_POWER.VBAT
- net GND: now also BAT1.-, R1.2, R3.1; no longer C12.2, C22.2, C23.2, C28.2, IC3.CLK, IC3.D, IC3.GND, Q3.S, Q4.S, R18.2, R22.2, R23.1, R24.2, R25.1, R3.2, S6.2, U$2.GND, U$2.P$4, U$2.P$5, U2.GND, U3.VSS
- net N$2: now also R1.1, S6.1; no longer R17.2, U3.STAT
- net N$7: now also LED1.C, R3.2; no longer R3.1, U3.PROG
- net RTC1: now also C9.1, Y2.2
- net RTC2: now also C6.1, Y2.1
- net VBUS: now also D3.C, U4.EN; no longer C12.1, C28.1, IC3.VCC, JP1.1, Q1.S, R6.1, R7.1
- net VBUS_IN: no longer C6.1, R25.2, U2.VCC, U3.VIN
Other:
- note added: "RTC"
- note removed: "Battery charging"
- note removed: "Battery detect"
- note removed: "Soft power"
- moved on the sheet: C1, C10, C11, C13, C14, C15, C18, C2, C26, C27, C35, C36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
