File: electronics/armwiz-board.sch (EAGLE design)
At the start: 62 parts, among them J1 MICRO-SDCARD-CONNECTOR-330006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, U1 STM32F10XRXT6, U4 MIC5219-3.3V, X1 FH12-12S-1S, Y1 16MHz

Commit message: Did some routing.
Parts:
- added J10, J13, J14, J15, J16, J17, J18, J8, J9: (no value), SparkFun-Connectors:M01SPRING-CONN
- added J19, J20, J21, J22, J23, J24, J25, J26, J3: (no value), SparkFun-Connectors:M01PTH_2MM
- added J7: (no value), SparkFun-Connectors:M06FEMALE_LOCK
Connections:
- net N$65 renamed SW_PWR
- new net N$10: J17.1, U1PORTA_H.PA9
- new net N$12: J18.1, U1PORTA_H.PA10
- net N$34: now also J8.1
- net N$40: now also J16.1
- net N$43: now also J7.6
- net N$45: now also J7.5
- net N$47: now also J7.4
- net N$51: now also J7.3
- net N$52: now also J7.2
- net N$53: now also J7.1
- net N$54: now also J19.1
- net N$57: now also J3.1
- net N$58: now also J20.1
- net N$59: now also J21.1
- net N$60: now also J22.1
- net N$61: now also J23.1
- net N$62: now also J24.1
- net N$63: now also J25.1
- net N$64: now also J26.1
- net N$66: now also J10.1
- net N$67: now also J13.1
- net N$68: now also J14.1
- net N$69: now also J15.1

Commit message: Basic layout done. Need to dome some details.
Parts:
- removed J14, J15, J17, J18: (no value), SparkFun-Connectors:M01SPRING-CONN
- removed J22: (no value), SparkFun-Connectors:M01PTH_2MM
- added J12, J27, J28, J29, J30, J31, J32, J33: (no value), SparkFun-Connectors:M01PTH
- added TP1: TPB1,27, testpad:TPB1,27
- J10, J13, J16, J8, J9: device SparkFun-Connectors:M01SPRING-CONN -> SparkFun-Connectors:M01PTH
- J11: device SparkFun-Connectors:M021X02_NO_SILK -> SparkFun-Connectors:M01PTH
- J19, J20, J21, J23, J24, J25, J26, J3: device SparkFun-Connectors:M01PTH_2MM -> SparkFun-Connectors:M01PTH
- J4, J5, J6: device SparkFun-Connectors:M08NO_SILK -> SparkFun-Connectors:M01PTH
- J7: device SparkFun-Connectors:M06FEMALE_LOCK -> SparkFun-Connectors:M01PTH
Connections:
- removed net N$10: J17.1, U1PORTA_H.PA9
- removed net N$101: J11.2
- removed net N$118: J11.1
- removed net N$12: J18.1, U1PORTA_H.PA10
- removed net N$2: R1.1, S6.1
- removed net N$29: U1PORTB_L.PB1
- removed net N$34: J8.1, U1PORTB_L.PB0
- removed net N$40: J16.1, U1PORTA_H.PA8
- removed net N$43: J7.6, U1PORTB_H.PB10
- removed net N$45: J7.5, U1PORTB_H.PB11
- removed net N$47: J7.4, U1PORTB_H.PB12
- removed net N$51: J7.3, U1PORTB_H.PB13
- removed net N$52: J7.2, U1PORTB_H.PB14
- removed net N$53: J7.1, U1PORTB_H.PB15
- removed net N$54: J19.1, U1PORTC_H.PC13
- removed net N$55: J6.1
- removed net N$56: J5.2
- removed net N$57: J3.1, U1PORTC_L.PC0
- removed net N$58: J20.1, U1PORTC_L.PC1
- removed net N$59: J21.1, U1PORTC_L.PC2
- removed net N$60: J22.1, U1PORTC_L.PC3
- removed net N$61: J23.1, U1PORTC_L.PC4
- removed net N$62: J24.1, U1PORTC_L.PC5
- removed net N$63: J25.1, U1PORTC_L.PC6
- removed net N$64: J26.1, U1PORTC_L.PC7
- removed net N$66: J10.1, U1PORTA_L.PA1
- removed net N$67: J13.1, U1PORTA_L.PA2
- removed net N$68: J14.1, U1PORTA_L.PA3
- removed net N$69: J15.1, U1PORTA_L.PA4
- removed net N$70: J4.3
- removed net N$71: J4.4
- removed net N$72: J4.5
- removed net N$73: J4.6
- removed net N$74: J4.7
- removed net N$75: J4.8
- removed net N$76: J4.1
- removed net N$77: J4.2
- removed net N$78: J5.3
- removed net N$79: J5.4
- removed net N$80: J5.5
- removed net N$81: J5.6
- removed net N$82: J5.7
- removed net N$83: J6.2
- removed net N$84: J5.1
- removed net N$85: J6.3
- removed net N$86: J6.4
- removed net N$87: J6.5
- removed net N$88: J6.6
- removed net N$89: J6.7
- removed net N$90: J6.8
- removed net N$91: J5.8
- new net PA1: J19.1, U1PORTA_L.PA1
- new net PA10: J23.1
- new net PA2: J3.1, U1PORTA_L.PA2
- new net PA3: J12.1, U1PORTA_L.PA3
- new net PA4: J5.1, U1PORTA_L.PA4
- new net PA8: TP1.TP, U1PORTA_H.PA8
- new net PA9: J25.1
- new net PB0: J6.1, U1PORTB_L.PB0
- new net PB1: J11.1, U1PORTB_L.PB1
- new net PB10: J24.1, U1PORTB_H.PB10
- new net PB11: J9.1, U1PORTB_H.PB11
- new net PB12: J26.1, U1PORTB_H.PB12
- new net PB13: J27.1, U1PORTB_H.PB13
- new net PB14: J28.1, U1PORTB_H.PB14
- new net PB15: J29.1, U1PORTB_H.PB15
- new net PC0: J16.1, U1PORTC_L.PC0
- new net PC1: J31.1, U1PORTC_L.PC1
- new net PC13: J30.1, U1PORTC_H.PC13
- new net PC2: J33.1, U1PORTC_L.PC2
- new net PC3: J7.1, U1PORTC_L.PC3
- new net PC4: J8.1, U1PORTC_L.PC4
- new net PC5: J32.1, U1PORTC_L.PC5
- new net PC6: J20.1, U1PORTC_L.PC6
- new net PC7: J21.1, U1PORTC_L.PC7
- net MISO1: now also J10.1
- net MOSI1: now also J13.1
- net SCLK1: now also J4.1
- net SW_D: now also U1PORTA_H.PA10
- net SW_E: now also U1PORTA_H.PA9
- net SW_PWR: now also R1.1, S6.1
Other:
- note removed: "Module Connector"
- moved on the sheet: J10, J13, J16, J19, J20, J21, J23, J24, J25, J26, J3, J8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

Commit message: Getting closer.
Parts:
- removed J16, J23, J30, J31: (no value), SparkFun-Connectors:M01PTH
Connections:
- removed net PA10: J23.1
- removed net PC0: J16.1, U1PORTC_L.PC0
- removed net PC1: J31.1, U1PORTC_L.PC1
- removed net PC13: J30.1, U1PORTC_H.PC13
- net SW_A: now also U1PORTC_L.PC1
- net SW_B: now also U1PORTC_L.PC0
- net SW_C: now also U1PORTC_H.PC13
Changed lines of the file:
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@@
 <part name="J20" library="SparkFun-Connectors" deviceset="M01" device="PTH"/>
 <part name="J21" library="SparkFun-Connectors" deviceset="M01" device="PTH"/>
-<part name="J23" library="SparkFun-Connectors" deviceset="M01" device="PTH"/>
 <part name="J24" library="SparkFun-Connectors" deviceset="M01" device="PTH"/>
 <part name="J25" library="SparkFun-Connectors" deviceset="M01" device="PTH"/>
@@
 <part name="J28" library="SparkFun-Connectors" deviceset="M01" device="PTH"/>
 <part name="J29" library="SparkFun-Connectors" deviceset="M01" device="PTH"/>
-<part name="J30" library="SparkFun-Connectors" deviceset="M01" device="PTH"/>
 <part name="J5" library="SparkFun-Connectors" deviceset="M01" device="PTH"/>
 <part name="J6" library="SparkFun-Connectors" deviceset="M01" device="PTH"/>
 <part name="J11" library="SparkFun-Connectors" deviceset="M01" device="PTH"/>
-<part name="J16" library="SparkFun-Connectors" deviceset="M01" device="PTH"/>
-<part name="J31" library="SparkFun-Connectors" deviceset="M01" device="PTH"/>
 <part name="J32" library="SparkFun-Connectors" deviceset="M01" device="PTH"/>
 <part name="J33" library="SparkFun-Connectors" deviceset="M01" device="PTH"/>
@@
 <instance part="J20" gate="G$1" x="142.24" y="48.26"/>
 <instance part="J21" gate="G$1" x="142.24" y="40.64"/>
-<instance part="J23" gate="G$1" x="162.56" y="78.74"/>
 <instance part="J24" gate="G$1" x="162.56" y="71.12"/>
 <instance part="J25" gate="G$1" x="142.24" y="25.4"/>
@@
 <instance part="J28" gate="G$1" x="162.56" y="40.64"/>
 <instance part="J29" gate="G$1" x="162.56" y="33.02"/>
-<instance part="J30" gate="G$1" x="162.56" y="25.4"/>
 <instance part="J5" gate="G$1" x="121.92" y="55.88"/>
 <instance part="J6" gate="G$1" x="121.92" y="48.26"/>
 <instance part="J11" gate="G$1" x="121.92" y="40.64"/>
-<instance part="J16" gate="G$1" x="121.92" y="33.02"/>
-<instance part="J31" gate="G$1" x="121.92" y="25.4"/>
 <instance part="J32" gate="G$1" x="142.24" y="55.88"/>
 <instance part="J33" gate="G$1" x="142.24" y="78.74"/>
@@
 </segment>
 <segment>
-<wire x1="91.44" y1="76.2" x2="93.98" y2="76.2" width="0.1524" layer="91"/>
-<label x="93.98" y="76.2" size="1.27" layer="95" xref="yes"/>
+<pinref part="U1" gate="PORTC_L" pin="PC0"/>
+<wire x1="27.94" y1="48.26" x2="30.48" y2="48.26" width="0.1524" layer="91"/>
+<label x="30.48" y="48.26" size="1.27" layer="95" xref="yes"/>
 </segment>
 </net>
@@
 </segment>
 <segment>
-<wire x1="91.44" y1="73.66" x2="93.98" y2="73.66" width="0.1524" layer="91"/>
-<label x="93.98" y="73.66" size="1.27" layer="95" xref="yes"/>
+<pinref part="U1" gate="PORTC_H" pin="PC13"/>
+<wire x1="63.5" y1="35.56" x2="66.04" y2="35.56" width="0.1524" layer="91"/>
+<label x="66.04" y="35.56" size="1.27" layer="95" xref="yes"/>
 </segment>
 </net>
@@
 </segment>
 <segment>
-<wire x1="91.44" y1="78.74" x2="93.98" y2="78.74" width="0.1524" layer="91"/>
-<label x="93.98" y="78.74" size="1.27" layer="95" xref="yes"/>
+<pinref part="U1" gate="PORTC_L" pin="PC1"/>
+<wire x1="27.94" y1="45.72" x2="30.48" y2="45.72" width="0.1524" layer="91"/>
+<label x="30.48" y="45.72" size="1.27" layer="95" xref="yes"/>
 </segment>
 </net>
@@
 </segment>
 </net>
-<net name="PC0" class="0">
-<segment>
-<pinref part="U1" gate="PORTC_L" pin="PC0"/>
-<wire x1="27.94" y1="48.26" x2="30.48" y2="48.26" width="0.1524" layer="91"/>
-<label x="30.48" y="48.26" size="1.27" layer="95" xref="yes"/>
-</segment>
-<segment>
-<label x="132.08" y="33.02" size="1.27" layer="95" xref="yes"/>
-<pinref part="J16" gate="G$1" pin="1"/>
-<wire x1="129.54" y1="33.02" x2="132.08" y2="33.02" width="0.1524" layer="91"/>
-</segment>
-</net>
-<net name="PC1" class="0">
-<segment>
-<pinref part="U1" gate="PORTC_L" pin="PC1"/>
-<wire x1="27.94" y1="45.72" x2="30.48" y2="45.72" width="0.1524" layer="91"/>
-<label x="30.48" y="45.72" size="1.27" layer="95" xref="yes"/>
-</segment>
-<segment>
-<label x="132.08" y="25.4" size="1.27" layer="95" xref="yes"/>
-<pinref part="J31" gate="G$1" pin="1"/>
-<wire x1="129.54" y1="25.4" x2="132.08" y2="25.4" width="0.1524" layer="91"/>
-</segment>
-</net>
 <net name="PC2" class="0">
 <segment>
@@
 </segment>
 </net>
-<net name="PC13" class="0">
-<segment>
-<pinref part="U1" gate="PORTC_H" pin="PC13"/>
-<wire x1="63.5" y1="35.56" x2="66.04" y2="35.56" width="0.1524" layer="91"/>
-<label x="66.04" y="35.56" size="1.27" layer="95" xref="yes"/>
-</segment>
-<segment>
-<pinref part="J30" gate="G$1" pin="1"/>
-<wire x1="170.18" y1="25.4" x2="172.72" y2="25.4" width="0.1524" layer="91"/>
-<label x="172.72" y="25.4" size="1.27" layer="95" xref="yes"/>
-</segment>
-</net>
 <net name="PB15" class="0">
 <segment>
@@
 </segment>
 </net>
-<net name="PA10" class="0">
-<segment>
-<pinref part="J23" gate="G$1" pin="1"/>
-<wire x1="170.18" y1="78.74" x2="172.72" y2="78.74" width="0.1524" layer="91"/>
-<label x="172.72" y="78.74" size="1.27" layer="95" xref="yes"/>
-</segment>
-</net>

Commit message: Moved some traces. Have a little more room now.
Parts:
- removed JP2: (no value), PaxInstruments-Connectors:M03X2PAX
- removed R30: 10k, SparkFun-Passives:RESISTOR-ARRAY0603-ARV
- added R17, R5, R6, R7: 10K, resistor:R-US_R0402
- added SJ1: (no value), SparkFun-Retired:SOLDERJUMPER_2WAYPASTE2&3
- added SJ2: (no value), SparkFun-Retired:SOLDERJUMPER_2WAYS
- added U$2: FOUR_LAYER_WARNING, SparkFun-Aesthetics:FOUR_LAYER_WARNING
Connections:
- net 3.3V: now also R17.1, R5.1, R6.1, R7.1, SJ1.1, SJ2.3; no longer JP2.1, JP2.2, R30A.1, R30B.1, R30C.1, R30D.1
- net BOOT0: now also SJ1.2; no longer JP2.4
- net BOOT1: now also SJ2.2; no longer JP2.3
- net GND: now also SJ1.3, SJ2.1; no longer JP2.5, JP2.6
- net SDIO_CLK: now also R7.2; no longer R13.2
- net SDIO_D0: now also R13.2; no longer R30C.2
- net SDIO_D1: now also R17.2; no longer R30D.2
- net SDIO_D2: now also R5.2; no longer R30A.2
- net SDIO_D3: now also R6.2; no longer R30B.2
Other:
- note added: "Breakout Header"
- moved on the sheet: BAT1, C14, C18, C35, C36, C6, C9, J1, J10, J11, J12, J13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
