File: electronics/armwiz-board.sch (EAGLE design)
At the start: 88 parts, among them J1 MICRO-SDCARD-CONNECTOR-330006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, J2 CORTEX_DEBUGSMD, U1 STM32F10XRXT6, U4 MIC5219-3.3V, X1 FH12-12S-1S, Y3 32.768kHz

Commit message: Really close now.
Parts:
- removed TP2, TP3, TP4: TPB1,27, testpad:TPB1,27
- added J15: Cortex Debug, SparkFun-Connectors:CORTEX_DEBUGSMD
- added J16: ST-Link v2, SparkFun-Connectors:M10X2
- added J17, J18: (no value), SparkFun-Connectors:M01NOSILK-KIT
- added R23: 100R, resistor:R-US_R0402
- added R24: 10K, resistor:R-US_R0402
- J14: device SparkFun-Connectors:M25PTH -> PaxInstruments-Connectors:M03X2PAX
Connections:
- new net AD_GND: J15.GND@3, J15.GND@5, J15.GNDDTCT, J16.10, J16.12, J16.14, J16.16, J16.18, J16.20, J16.4, J16.6, J16.8
- new net AD_NRST: J15.NRESET, J16.15
- new net AD_SWDCLK: J15.SWDCLK/TCK, J16.9
- new net AD_SWDIO: J15.SWDIO/TMS, J16.7
- new net AD_SWO: J15.SWO/TDO, J16.13
- new net AD_TDI: J15.NC/TDI, J16.5
- new net AD_VCC: J15.VCC, J16.1
- new net N$12: J2.SWO/TDO, R23.2
- net 3.3V: now also J14.1, J18.1, R24.2
- net BOOT0: now also J17.1; no longer TP2.TP
- net GND: now also J14.3; no longer J2.KEY
- net NRST: now also J14.5
- net SWDCLK: now also J14.2
- net SWDIO: now also J14.4
- net SWO: now also J14.6, R23.1, R24.1; no longer J2.SWO/TDO
- net USART1_RX: no longer TP3.TP
- net USART1_TX: no longer TP4.TP
Other:
- note added: "Cortex Debug Adapter"
- note added: "Indicator LEDs"
- moved on the sheet: C3, C35, C36, J26, J27, LED1, LED2, R19, R22, R28, R3, SJ2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

Commit message: Four more wires.
Parts:
- added J22: (no value), SparkFun-Connectors:M01PTH
Connections:
- net PC1: now also J22.1
Changed lines of the file:
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@@
 <part name="J18" library="SparkFun-Connectors" deviceset="M01" device="NOSILK-KIT"/>
 <part name="P+5" library="SparkFun" deviceset="3.3V" device=""/>
+<part name="J22" library="SparkFun-Connectors" deviceset="M01" device="PTH"/>
 </parts>
 <sheets>
@@
 <instance part="J18" gate="G$1" x="360.68" y="215.9"/>
 <instance part="P+5" gate="G$1" x="368.3" y="218.44"/>
+<instance part="J22" gate="G$1" x="167.64" y="40.64"/>
 </instances>
 <busses>
@@
 <label x="30.48" y="45.72" size="1.27" layer="95" xref="yes"/>
 </segment>
-</net>
+<segment>
+<pinref part="J22" gate="G$1" pin="1"/>
+<wire x1="175.26" y1="40.64" x2="177.8" y2="40.64" width="0.1524" layer="91"/>
+<label x="177.8" y="40.64" size="1.27" layer="95" xref="yes"/>
+</segment>
+</net>
