File: electronics/armwiz-board.sch (EAGLE design)
At the start: 79 parts, among them J1 MICROSD, J2 CORTEX_DEBUGSMD, U1 STM32F10XRXT6, U4 MIC5219-3.3V, X2 M12_BOTTOM_CONTACTS_FPC_1MM, Y1 32.768kHz, Y3 32.768kHz

Commit message: Crazy routing work.
Connections:
- removed net PA1: U1PORTA_L.PA1
- removed net PC2: U1PORTC_L.PC2
- removed net PC3: U1PORTC_L.PC3
- net SW_A: now also U1PORTA_L.PA1
- net SW_B: now also U1PORTC_L.PC3
- net SW_C: now also U1PORTC_L.PC2
Changed lines of the file:
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@@
 </segment>
 </net>
-<net name="GND" class="0">
+<net name="GND" class="5">
 <segment>
 <wire x1="248.92" y1="96.52" x2="243.84" y2="96.52" width="0.1524" layer="91"/>
@@
 <label x="165.1" y="137.16" size="1.27" layer="95" xref="yes"/>
 </segment>
+<segment>
+<pinref part="U1" gate="PORTC_L" pin="PC3"/>
+<wire x1="27.94" y1="38.1" x2="30.48" y2="38.1" width="0.1524" layer="91"/>
+<label x="30.48" y="38.1" size="1.27" layer="95" xref="yes"/>
+</segment>
 </net>
 <net name="SW_C" class="0">
@@
 <wire x1="152.4" y1="17.78" x2="157.48" y2="17.78" width="0.1524" layer="91"/>
 <label x="160.02" y="17.78" size="1.27" layer="95" xref="yes"/>
-<label x="165.1" y="134.62" size="1.27" layer="95" xref="yes"/>
 <pinref part="R12" gate="G$1" pin="2"/>
 <wire x1="157.48" y1="17.78" x2="160.02" y2="17.78" width="0.1524" layer="91"/>
 <wire x1="157.48" y1="25.4" x2="157.48" y2="17.78" width="0.1524" layer="91"/>
 <junction x="157.48" y="17.78"/>
+</segment>
+<segment>
+<pinref part="U1" gate="PORTC_L" pin="PC2"/>
+<wire x1="27.94" y1="40.64" x2="30.48" y2="40.64" width="0.1524" layer="91"/>
+<label x="30.48" y="40.64" size="1.27" layer="95" xref="yes"/>
 </segment>
 </net>
@@
 <label x="160.02" y="22.86" size="1.27" layer="95" xref="yes"/>
 <label x="165.1" y="139.7" size="1.27" layer="95" xref="yes"/>
+</segment>
+<segment>
+<pinref part="U1" gate="PORTA_L" pin="PA1"/>
+<wire x1="27.94" y1="93.98" x2="30.48" y2="93.98" width="0.1524" layer="91"/>
+<label x="30.48" y="93.98" size="1.27" layer="95" xref="yes"/>
 </segment>
 </net>
@@
 </segment>
 </net>
-<net name="PA1" class="0">
-<segment>
-<pinref part="U1" gate="PORTA_L" pin="PA1"/>
-<wire x1="27.94" y1="93.98" x2="30.48" y2="93.98" width="0.1524" layer="91"/>
-<label x="30.48" y="93.98" size="1.27" layer="95" xref="yes"/>
-</segment>
-</net>
 <net name="USART2_TX" class="0">
 <segment>
@@
 </segment>
 </net>
-<net name="PC2" class="0">
-<segment>
-<pinref part="U1" gate="PORTC_L" pin="PC2"/>
-<wire x1="27.94" y1="40.64" x2="30.48" y2="40.64" width="0.1524" layer="91"/>
-<label x="30.48" y="40.64" size="1.27" layer="95" xref="yes"/>
-</segment>
-</net>
-<net name="PC3" class="0">
-<segment>
-<pinref part="U1" gate="PORTC_L" pin="PC3"/>
-<wire x1="27.94" y1="38.1" x2="30.48" y2="38.1" width="0.1524" layer="91"/>
-<label x="30.48" y="38.1" size="1.27" layer="95" xref="yes"/>
-</segment>
-</net>

Commit message: Routed. Passes DRC. Added a thermocouple module.
Parts:
- removed J25: (no value), PaxInstruments-Connectors:M03X2PAX
- removed LED1, LED2: GREEN, SparkFun-LED:LED0603
- removed R17, R21, R5, R6: 10K, PaxInstruments-RCL:R0402_10K
- removed R22: 360R, PaxInstruments-RCL:R0402_360R
- removed SJ2: (no value), SparkFun-Retired:SOLDERJUMPER_2WAYS
- added C22, C23: 100nF, PaxInstruments-RCL:C0402_100NF
- added C24: 1uF, PaxInstruments-RCL:C0402_1UF
- added IC1: MCP3424, PaxInstruments-DigitalIC:MCP3424
- added MODULE5, MODULE6: PI-module-male, PaxInstruments-Connectors:PAX_MODULE_EDGE_MALE_MODULE
- added TP1, TP2, TP3, TP4: (no value), PaxInstruments-Connectors:M01_TH
- added TP7: (no value), PaxInstruments-Connectors:M01_PAD_1MM
- added U$4: MCP9800A0, PaxInstruments-DigitalIC:MCP9800A0
- added U$7: THERMOCOUPLE_MINI_INSIDE, PaxInstruments-Connectors:THERMOCOUPLE_MINI_INSIDE
- added U$8: 0.25 in, PaxInstruments-Aesthetics:PAX-LOGO_0.25IN
- J1: value MICROSD -> SD_MICRO_SDIO_1BIT; device PaxInstruments-Connectors:MICROSD -> PaxInstruments-Connectors:SD_MICRO_SDIO_1BIT; MPN ST-TF-003A -> (none)
- R3: value 360R -> 10K; device PaxInstruments-RCL:R0402_360R -> PaxInstruments-RCL:R0402_10K
Connections:
- removed net (BOOT1): SJ2.2, U1PORTB_L.PB2
- removed net LED2: LED2.A
- removed net N$11: LED2.C, R22.1
- removed net N$51: MODULE3.GPIO1
- removed net N$57: MODULE1.GPIO1
- removed net N$68: MODULE2.GPIO0
- removed net N$69: MODULE2.GPIO1
- removed net N$7: LED1.C, R3.1
- removed net N$74: MODULE4.GPIO0
- removed net N$75: MODULE4.GPIO1
- removed net PA8: U1PORTA_H.PA8
- removed net PB0: U1PORTB_L.PB0
- removed net PB1: U1PORTB_L.PB1
- removed net PC0: U1PORTC_L.PC0
- removed net PC4: U1PORTC_L.PC4
- removed net PC5: U1PORTC_L.PC5
- removed net PC7: U1PORTC_L.PC7
- removed net SDIO_D1: J1.SDIO_D1, R17.1, U1PORTC_H.PC9
- removed net SDIO_D2: J1.SDIO_D2, R5.1, U1PORTC_H.PC10
- removed net SDIO_D3: J1.SDIO_D3, R6.1, U1PORTC_H.PC11
- removed net SW_E: R16.2, S5.2
- new net 3.3V_1: C22.2, C23.2, C24.2, IC1.VDD, MODULE5.3V3, TP3.P$1, U$4.1
- new net 3.3V_2: MODULE6.3V3
- new net GND_1: C22.1, C23.1, C24.1, IC1.A0, IC1.GND, MODULE5.GND, TP4.P$1, U$4.2
- new net GND_2: MODULE6.GND
- new net MOD1_GPIO1: MODULE1.GPIO1, U1PORTC_L.PC4
- new net MOD2_GPIO0: MODULE2.GPIO0, U1PORTA_L.PA1
- new net MOD2_GPIO1: MODULE2.GPIO1, U1PORTC_L.PC3
- new net MOD3_GPIO1: MODULE3.GPIO1, U1PORTC_L.PC2
- new net MOD4_GPIO0: MODULE4.GPIO0, U1PORTC_L.PC5
- new net MOD4_GPIO1: MODULE4.GPIO1, U1PORTB_L.PB1
- new net N$25: IC1.CH1-, U$7.P$1
- new net N$26: IC1.CH1+, U$7.P$2
- new net SCL_1: IC1.SCL, MODULE5.I2C_SCL, TP2.P$1, U$4.4
- new net SDA_1: IC1.SDA, MODULE5.I2C_SDA, TP1.P$1, U$4.5
- new net SW_E_(BOOT1): R16.2, S5.2, U1PORTB_L.PB2
- net 3.3V: no longer J25.1, LED1.A, R17.2, R5.2, R6.2, SJ2.3
- net BOOT0: now also R3.2; no longer R21.2
- net GND: now also R3.1; no longer J25.5, MODULE1.KEY, MODULE2.KEY, MODULE3.KEY, MODULE4.KEY, R21.1, R22.2, R3.2, SJ2.1
- net LCD_A0_(GPIO): now also U1PORTC_L.PC0; no longer U1PORTC_L.PC1
- net PC6: now also TP7.P$1
- net SD_DETECT: now also U1PORTC_L.PC1
- net SW_A: now also U1PORTC_H.PC11; no longer U1PORTA_L.PA1
- net SW_B: now also U1PORTC_H.PC10; no longer U1PORTC_L.PC3
- net SW_C: now also U1PORTC_L.PC7; no longer U1PORTC_L.PC2
- net SW_D: now also U1PORTA_H.PA8
- net USART1_RX: now also J2.NC/TDI; no longer J25.2
- net USART1_TX: now also J2.SWO/TDO; no longer J25.4
- net VBAT_1/2: now also U1PORTB_L.PB0
- net VBUS: now also U1PORTC_H.PC9
Other:
- note added: "Module 1: Thermocouple"
- note added: "Module 2"
- note removed: "Boot config"
- note removed: "Indicator LEDs"
- note removed: "Serial Header"
- moved on the sheet: C3, R2, R3, R4, U1RESET

Commit message: Changed serial pins on Cortex header. Added SWO to Cortex header. Added TODO notes to schematic.
Connections:
- removed net LCD_SCK_(SPI3_SCK): U1PORTB_L.PB3, X2.7
- new net LCD_SCK_(SPI3_SCK_SWO): J2.SWO/TDO, U1PORTB_L.PB3, X2.7
- net USART1_RX: now also J2.KEY; no longer J2.NC/TDI
- net USART1_TX: now also J2.NC/TDI; no longer J2.SWO/TDO
Other:
- note added: "NOTES - Connect PC6 to somthing useful - Connect BOOT0 to something useful"
- moved on the sheet: BAT1, C1, C10, C11, C12, C13, C14, C15, C16, C17, C18, C19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
