File: electronics/versions/labwiz-board-v0.1.1/armwiz-board.brd (EAGLE design)
At the start: 99.1 x 51.5 mm, 100 parts, among them J1 MICRO-SDCARD-CONNECTOR-330006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, J15 Cortex Debug, J16 ST-Link v2, J2 CORTEX_DEBUGSMD, U1 STM32F10XRXT6, U4 MIC5219-3.3V, X1 FH12-12S-1S, Y3 32.768kHz

Commit message: Added pin docs to silk.
Other:
- board text added: "MISO1"
- board text added: "MOSI1"
- board text added: "PA1"
- board text added: "PA2"
- board text added: "PA3"
- board text added: "PA4"
- board text added: "PB0"
- board text added: "PB1"
- board text added: "PB10"
- board text added: "PC0"
- board text added: "PC1"
- board text added: "PC13"
- board text added: "PC2"
- board text added: "PC3"
- board text added: "PC4"
- board text added: "SCLK1"
Changed lines of the file:
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@@
 <setting verticaltext="up"/>
 </settings>
-<grid distance="0.25" unitdist="mm" unit="mm" style="lines" multiple="1" display="yes" altdistance="0.05" altunitdist="mil" altunit="inch"/>
+<grid distance="0.5" unitdist="mm" unit="mm" style="lines" multiple="1" display="yes" altdistance="0.05" altunitdist="mil" altunit="inch"/>
 <layers>
 <layer number="1" name="Top" color="4" fill="1" visible="yes" active="yes"/>
@@
 <wire x1="16.25" y1="22.5" x2="15.26" y2="22.5" width="0.127" layer="20"/>
 <wire x1="15.26" y1="23.5" x2="16.25" y2="23.5" width="0.127" layer="20"/>
+<text x="18.5" y="22" size="1.778" layer="47" rot="R90">MOSI1</text>
+<text x="21" y="22" size="1.778" layer="47" rot="R90">MISO1</text>
+<text x="23.5" y="22" size="1.778" layer="47" rot="R90">SCLK1</text>
+<text x="26" y="22" size="1.778" layer="47" rot="R90">PA4</text>
+<text x="29" y="22" size="1.778" layer="47" rot="R90">PB0</text>
+<text x="31.5" y="22" size="1.778" layer="47" rot="R90">PA3</text>
+<text x="34" y="22" size="1.778" layer="47" rot="R90">PA2</text>
+<text x="36.5" y="22" size="1.778" layer="47" rot="R90">PA1</text>
+<text x="39" y="22" size="1.778" layer="47" rot="R90">PB10</text>
+<text x="41.5" y="22" size="1.778" layer="47" rot="R90">PB1</text>
+<text x="44" y="22" size="1.778" layer="47" rot="R90">PC3</text>
+<text x="46.5" y="22" size="1.778" layer="47" rot="R90">PC2</text>
+<text x="49" y="22" size="1.778" layer="47" rot="R90">PC1</text>
+<text x="51.5" y="22" size="1.778" layer="47" rot="R90">PC0</text>
+<text x="54" y="22" size="1.778" layer="47" rot="R90">PC4</text>
+<text x="57" y="22" size="1.778" layer="47" rot="R90">PC13</text>
 </plain>
 <attributes>
