File: electronics/extras/labwiz-module_full_breakout/labwiz-module_full_breakout.brd (EAGLE design)
At the start: 66 x 33.2 mm, 8 parts

Commit message: Moved modules into folders.
Parts:
- moved J1 1.00 mm to (1.54, 25.4)
- moved J2 1.00 mm to (1.54, 27.9)
- moved J3 1.00 mm to (1.54, 30.5)
- moved J4 1.00 mm to (1.54, 22.9)
- moved MODULE5 1.00 mm to (14.0, 1.00)
- moved MODULE6 1.00 mm to (30.0, 1.00)
- moved MODULE7 1.00 mm to (46.0, 1.00)
- moved MODULE8 1.00 mm to (62.0, 1.00)
Other:
- board size 66 x 33.2 mm -> 64 x 33.2 mm
