File: electronics/extras/labwiz-module_servo_dual/labwiz-module_servo_dual.sch (EAGLE design)
At the start: 8 parts, among them U1 NCP1402

Commit message: Small changes. Not sure what.
Parts:
- removed C2: 68uF, SparkFun:CAP_POL3528
- added C3: 68uF, PaxInstruments-RCL:CAPACITOR_FIXED_0603
- C1: device SparkFun:CAP_POL1206 -> PaxInstruments-RCL:CAPACITOR_FIXED_10UF_0603
Connections:
- removed net 3.3V: C1.+, L1.1, MODULE5.3V3
- removed net CANH: MODULE5.CAN_TX
- removed net CANL: MODULE5.CAN_RX
- removed net I2C_SCL: MODULE5.I2C_SCL
- removed net I2C_SDA: MODULE5.I2C_SDA
- removed net SPI_MISO: MODULE5.SPI_MISO
- removed net SPI_MOSI: MODULE5.SPI_MOSI
- removed net SPI_SCK: MODULE5.SPI_SCK
- removed net USART_RX: MODULE5.UART_RX
- removed net USART_TX: MODULE5.UART_TX
- new net VBUS: C1.2, L1.1, MODULE5.VBUS
- net 5V: now also C3.2; no longer C2.+
- net GND: now also C1.1, C3.1, MODULE5.GND_A, MODULE5.GND_B; no longer C1.-, C2.-, MODULE5.GND
- net SERVO1: now also MODULE5.GPIO1; no longer MODULE5.GPIO0
- net SERVO2: now also MODULE5.GPIO2; no longer MODULE5.GPIO1
Changed lines of the file:
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@@
 <part name="FRAME1" library="SparkFun" deviceset="FRAME-A3" device=""/>
 <part name="MODULE5" library="PaxInstruments-Connectors" deviceset="PAX_MODULE" device="_EDGE_MALE_MODULE" value="PI-module-male"/>
-<part name="SUPPLY1" library="PaxInstruments-Aesthetics" deviceset="SYM_VCC" device="" technology="3.3V" value="3.3V"/>
 <part name="GND1" library="PaxInstruments-Aesthetics" deviceset="GND" device="" value="GND"/>
 <part name="J1" library="SparkFun-Connectors" deviceset="M03" device="1X03_SMD_RA_MALE_POST_SMALLEST"/>
@@
 <part name="U1" library="SparkFun" deviceset="V_REG_NCP1400" device="SOT23-5" value="NCP1402"/>
 <part name="D1" library="SparkFun" deviceset="DIODE" device="SMA" value="MBRA140"/>
-<part name="C1" library="SparkFun" deviceset="CAP_POL" device="1206" value="10uF"/>
-<part name="C2" library="SparkFun" deviceset="CAP_POL" device="3528" value="68uF"/>
 <part name="L1" library="SparkFun" deviceset="INDUCTOR" device="CR54" value="47uH"/>
 <part name="GND5" library="SparkFun" deviceset="GND" device=""/>
@@
 <part name="SUPPLY3" library="SparkFun-Aesthetics" deviceset="5V" device=""/>
 <part name="SUPPLY4" library="SparkFun-Aesthetics" deviceset="5V" device=""/>
-<part name="SUPPLY5" library="PaxInstruments-Aesthetics" deviceset="SYM_VCC" device="" technology="3.3V" value="3.3V"/>
+<part name="GND4" library="PaxInstruments-Aesthetics" deviceset="GND" device="" value="GND"/>
+<part name="C1" library="PaxInstruments-RCL" deviceset="CAPACITOR_FIXED" device="_0603" technology="_10UF" value="10uF"/>
+<part name="C3" library="PaxInstruments-RCL" deviceset="CAPACITOR_FIXED" device="_0603" value="68uF"/>
 </parts>
 <sheets>
@@
 <instance part="FRAME1" gate="G$1" x="0" y="0"/>
 <instance part="MODULE5" gate="G$1" x="48.26" y="215.9"/>
-<instance part="SUPPLY1" gate="G$1" x="27.94" y="236.22"/>
 <instance part="GND1" gate="G$1" x="66.04" y="233.68" rot="R90"/>
 <instance part="J1" gate="J$1" x="124.46" y="238.76"/>
@@
 <attribute name="VALUE" x="142.24" y="185.6486" size="1.778" layer="96"/>
 </instance>
-<instance part="C1" gate="G$1" x="104.14" y="170.18"/>
-<instance part="C2" gate="G$1" x="162.56" y="170.18"/>
 <instance part="L1" gate="G$1" x="116.84" y="175.26" smashed="yes" rot="R90">
 <attribute name="NAME" x="114.3" y="177.8" size="1.778" layer="95"/>
@@
 <instance part="SUPPLY3" gate="G$1" x="142.24" y="218.44" rot="R270"/>
 <instance part="SUPPLY4" gate="G$1" x="172.72" y="180.34"/>
-<instance part="SUPPLY5" gate="G$1" x="96.52" y="180.34"/>
+<instance part="GND4" gate="G$1" x="66.04" y="218.44" rot="R90"/>
+<instance part="C1" gate="G$1" x="104.14" y="170.18"/>
+<instance part="C3" gate="G$1" x="162.56" y="167.64"/>
 </instances>
 <busses>
 </busses>
 <nets>
-<net name="CANL" class="0">
-<segment>
-<pinref part="MODULE5" gate="G$1" pin="CAN_RX"/>
-<wire x1="63.5" y1="231.14" x2="66.04" y2="231.14" width="0.1524" layer="91"/>
-<label x="66.04" y="231.14" size="1.27" layer="95" xref="yes"/>
-</segment>
-</net>
-<net name="CANH" class="0">
-<segment>
-<pinref part="MODULE5" gate="G$1" pin="CAN_TX"/>
-<wire x1="63.5" y1="228.6" x2="66.04" y2="228.6" width="0.1524" layer="91"/>
-<label x="66.04" y="228.6" size="1.27" layer="95" xref="yes"/>
-</segment>
-</net>
-<net name="I2C_SDA" class="0">
-<segment>
-<pinref part="MODULE5" gate="G$1" pin="I2C_SDA"/>
-<wire x1="63.5" y1="226.06" x2="66.04" y2="226.06" width="0.1524" layer="91"/>
-<label x="66.04" y="226.06" size="1.27" layer="95" xref="yes"/>
-</segment>
-</net>
-<net name="I2C_SCL" class="0">
-<segment>
-<pinref part="MODULE5" gate="G$1" pin="I2C_SCL"/>
-<wire x1="63.5" y1="223.52" x2="66.04" y2="223.52" width="0.1524" layer="91"/>
-<label x="66.04" y="223.52" size="1.27" layer="95" xref="yes"/>
-</segment>
-</net>
-<net name="USART_RX" class="0">
-<segment>
-<pinref part="MODULE5" gate="G$1" pin="UART_RX"/>
-<wire x1="63.5" y1="220.98" x2="66.04" y2="220.98" width="0.1524" layer="91"/>
-<label x="66.04" y="220.98" size="1.27" layer="95" xref="yes"/>
-</segment>
-</net>
-<net name="USART_TX" class="0">
-<segment>
-<pinref part="MODULE5" gate="G$1" pin="UART_TX"/>
-<wire x1="63.5" y1="218.44" x2="66.04" y2="218.44" width="0.1524" layer="91"/>
-<label x="66.04" y="218.44" size="1.27" layer="95" xref="yes"/>
-</segment>
-</net>
-<net name="SPI_SCK" class="0">
-<segment>
-<pinref part="MODULE5" gate="G$1" pin="SPI_SCK"/>
-<wire x1="33.02" y1="226.06" x2="30.48" y2="226.06" width="0.1524" layer="91"/>
-<label x="30.48" y="226.06" size="1.27" layer="95" rot="R180" xref="yes"/>
-</segment>
-</net>
-<net name="SPI_MISO" class="0">
-<segment>
-<pinref part="MODULE5" gate="G$1" pin="SPI_MISO"/>
-<wire x1="33.02" y1="228.6" x2="30.48" y2="228.6" width="0.1524" layer="91"/>
-<label x="30.48" y="228.6" size="1.27" layer="95" rot="R180" xref="yes"/>
-</segment>
-</net>
-<net name="SPI_MOSI" class="0">
-<segment>
-<pinref part="MODULE5" gate="G$1" pin="SPI_MOSI"/>
-<wire x1="33.02" y1="231.14" x2="30.48" y2="231.14" width="0.1524" layer="91"/>
-<label x="30.48" y="231.14" size="1.27" layer="95" rot="R180" xref="yes"/>
-</segment>
-</net>
-<net name="3.3V" class="0">
-<segment>
-<pinref part="MODULE5" gate="G$1" pin="3V3"/>
-<wire x1="33.02" y1="233.68" x2="27.94" y2="233.68" width="0.1524" layer="91"/>
-<pinref part="SUPPLY1" gate="G$1" pin="3.3V"/>
-<wire x1="27.94" y1="233.68" x2="27.94" y2="236.22" width="0.1524" layer="91"/>
-</segment>
-<segment>
-<wire x1="109.22" y1="175.26" x2="104.14" y2="175.26" width="0.1524" layer="91"/>
-<wire x1="104.14" y1="175.26" x2="104.14" y2="172.72" width="0.1524" layer="91"/>
-<junction x="104.14" y="175.26"/>
-<pinref part="L1" gate="G$1" pin="1"/>
-<pinref part="C1" gate="G$1" pin="+"/>
-<pinref part="SUPPLY5" gate="G$1" pin="3.3V"/>
-<wire x1="96.52" y1="175.26" x2="104.14" y2="175.26" width="0.1524" layer="91"/>
-<wire x1="96.52" y1="180.34" x2="96.52" y2="175.26" width="0.1524" layer="91"/>
-</segment>
-</net>
 <net name="GND" class="0">
 <segment>
-<pinref part="MODULE5" gate="G$1" pin="GND"/>
+<pinref part="MODULE5" gate="G$1" pin="GND_A"/>
 <pinref part="GND1" gate="G$1" pin="GND"/>
 <wire x1="63.5" y1="233.68" x2="66.04" y2="233.68" width="0.1524" layer="91"/>
@@
 <segment>
 <wire x1="162.56" y1="165.1" x2="162.56" y2="162.56" width="0.1524" layer="91"/>
-<pinref part="C2" gate="G$1" pin="-"/>
 <pinref part="GND7" gate="1" pin="GND"/>
+<pinref part="C3" gate="G$1" pin="1"/>
 </segment>
 <segment>
@@
 </segment>
 <segment>
-<wire x1="104.14" y1="165.1" x2="104.14" y2="162.56" width="0.1524" layer="91"/>
-<pinref part="C1" gate="G$1" pin="-"/>
+<wire x1="104.14" y1="167.64" x2="104.14" y2="162.56" width="0.1524" layer="91"/>
 <pinref part="GND5" gate="1" pin="GND"/>
+<pinref part="C1" gate="G$1" pin="1"/>
+</segment>
+<segment>
+<pinref part="MODULE5" gate="G$1" pin="GND_B"/>
+<pinref part="GND4" gate="G$1" pin="GND"/>
+<wire x1="63.5" y1="218.44" x2="66.04" y2="218.44" width="0.1524" layer="91"/>
 </segment>
 </net>
@@
 </segment>
 <segment>
-<pinref part="MODULE5" gate="G$1" pin="GPIO0"/>
+<pinref part="MODULE5" gate="G$1" pin="GPIO1"/>
 <wire x1="33.02" y1="223.52" x2="30.48" y2="223.52" width="0.1524" layer="91"/>
 <label x="30.48" y="223.52" size="1.27" layer="95" rot="R180" xref="yes"/>
@@
 </segment>
 <segment>
-<pinref part="MODULE5" gate="G$1" pin="GPIO1"/>
+<pinref part="MODULE5" gate="G$1" pin="GPIO2"/>
 <wire x1="33.02" y1="220.98" x2="30.48" y2="220.98" width="0.1524" layer="91"/>
 <label x="30.48" y="220.98" size="1.27" layer="95" rot="R180" xref="yes"/>
@@
 <wire x1="152.4" y1="185.42" x2="152.4" y2="175.26" width="0.1524" layer="91"/>
 <wire x1="152.4" y1="175.26" x2="162.56" y2="175.26" width="0.1524" layer="91"/>
-<wire x1="162.56" y1="175.26" x2="162.56" y2="172.72" width="0.1524" layer="91"/>
+<wire x1="162.56" y1="175.26" x2="162.56" y2="170.18" width="0.1524" layer="91"/>
 <wire x1="162.56" y1="175.26" x2="172.72" y2="175.26" width="0.1524" layer="91"/>
 <junction x="152.4" y="175.26"/>
@@
 <pinref part="U1" gate="G$1" pin="OUT"/>
 <pinref part="D1" gate="G$1" pin="C"/>
-<pinref part="C2" gate="G$1" pin="+"/>
+<pinref part="C3" gate="G$1" pin="2"/>
 </segment>
 <segment>
@@
 </segment>
 </net>
+<net name="VBUS" class="0">
+<segment>
+<pinref part="MODULE5" gate="G$1" pin="VBUS"/>
+<wire x1="63.5" y1="226.06" x2="66.04" y2="226.06" width="0.1524" layer="91"/>
+<label x="66.04" y="226.06" size="1.27" layer="95" xref="yes"/>
+</segment>
+<segment>
+<wire x1="109.22" y1="175.26" x2="104.14" y2="175.26" width="0.1524" layer="91"/>
+<junction x="104.14" y="175.26"/>
+<pinref part="L1" gate="G$1" pin="1"/>
+<wire x1="96.52" y1="175.26" x2="104.14" y2="175.26" width="0.1524" layer="91"/>
+<label x="96.52" y="175.26" size="1.27" layer="95" rot="R180" xref="yes"/>
+<pinref part="C1" gate="G$1" pin="2"/>
+<wire x1="104.14" y1="175.26" x2="104.14" y2="172.72" width="0.1524" layer="91"/>
+</segment>
+</net>
