File: electronics/extras/labwiz-module_single_breakout/labwiz-module_single_breakout.brd (EAGLE design)
At the start: 16 x 33.2 mm, 1 part

Commit message: Updated .gitignore. Comitting unknown schematic updates.
Changed lines of the file:
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@@
 <setting verticaltext="up"/>
 </settings>
-<grid distance="1" unitdist="mm" unit="mm" style="lines" multiple="1" display="yes" altdistance="0.05" altunitdist="mil" altunit="inch"/>
+<grid distance="0.05" unitdist="mm" unit="mm" style="lines" multiple="1" display="yes" altdistance="0.05" altunitdist="mil" altunit="inch"/>
 <layers>
 <layer number="1" name="Top" color="4" fill="1" visible="yes" active="yes"/>
@@
 <text x="12" y="2" size="1.25" layer="22" rot="MR90" align="center-left">USART2_RX</text>
 <text x="14" y="2" size="1.25" layer="22" rot="MR90" align="center-left">USART2_TX</text>
+<polygon width="0" layer="49">
+<vertex x="-0.7" y="0"/>
+<vertex x="2.6" y="0"/>
+<vertex x="2.6" y="0.7" curve="-90"/>
+<vertex x="3" y="1.1" curve="-90"/>
+<vertex x="3.4" y="0.7"/>
+<vertex x="3.4" y="0"/>
+<vertex x="12.6" y="0"/>
+<vertex x="12.6" y="0.7" curve="-90"/>
+<vertex x="13" y="1.1" curve="-90"/>
+<vertex x="13.4" y="0.7"/>
+<vertex x="13.4" y="0"/>
+<vertex x="16.7" y="0"/>
+<vertex x="16.7" y="24.75" curve="-90"/>
+<vertex x="15.7" y="25.75" curve="-90"/>
+<vertex x="16.7" y="26.75"/>
+<vertex x="16.7" y="31.25"/>
+<vertex x="-0.7" y="31.25"/>
+<vertex x="-0.7" y="26.75" curve="-90"/>
+<vertex x="0.3" y="25.75" curve="-90"/>
+<vertex x="-0.7" y="24.75"/>
+</polygon>
 </plain>
 <attributes>
