File: electronics/extras/labwiz-module_single_breakout/labwiz-module_single_breakout.sch (EAGLE design)
At the start: 1 part

Commit message: Updated .gitignore. Comitting unknown schematic updates.
Connections:
- net 3.3V: now also MODULE5.3V3_A; no longer MODULE5.3V3
- net CANH: now also MODULE5.UART_TX; no longer MODULE5.CAN_TX
- net CANL: now also MODULE5.UART_RX; no longer MODULE5.CAN_RX
- net GND: now also MODULE5.GND_A; no longer MODULE5.GND
- net GPIO0: now also MODULE5.GPIO1; no longer MODULE5.GPIO0
- net GPIO1: now also MODULE5.GPIO2; no longer MODULE5.GPIO1
- net I2C_SDA: now also MODULE5.VBUS; no longer MODULE5.I2C_SDA
- net USART_RX: now also MODULE5.I2C_SDA; no longer MODULE5.UART_RX
- net USART_TX: now also MODULE5.GND_B; no longer MODULE5.UART_TX
Changed lines of the file:
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@@
 <net name="CANL" class="0">
 <segment>
-<pinref part="MODULE5" gate="G$1" pin="CAN_RX"/>
+<pinref part="MODULE5" gate="G$1" pin="UART_RX"/>
 <wire x1="63.5" y1="231.14" x2="66.04" y2="231.14" width="0.1524" layer="91"/>
 <label x="66.04" y="231.14" size="1.27" layer="95" xref="yes"/>
@@
 <net name="CANH" class="0">
 <segment>
-<pinref part="MODULE5" gate="G$1" pin="CAN_TX"/>
+<pinref part="MODULE5" gate="G$1" pin="UART_TX"/>
 <wire x1="63.5" y1="228.6" x2="66.04" y2="228.6" width="0.1524" layer="91"/>
 <label x="66.04" y="228.6" size="1.27" layer="95" xref="yes"/>
@@
 <net name="I2C_SDA" class="0">
 <segment>
-<pinref part="MODULE5" gate="G$1" pin="I2C_SDA"/>
+<pinref part="MODULE5" gate="G$1" pin="VBUS"/>
 <wire x1="63.5" y1="226.06" x2="66.04" y2="226.06" width="0.1524" layer="91"/>
 <label x="66.04" y="226.06" size="1.27" layer="95" xref="yes"/>
@@
 <net name="USART_RX" class="0">
 <segment>
-<pinref part="MODULE5" gate="G$1" pin="UART_RX"/>
+<pinref part="MODULE5" gate="G$1" pin="I2C_SDA"/>
 <wire x1="63.5" y1="220.98" x2="66.04" y2="220.98" width="0.1524" layer="91"/>
 <label x="66.04" y="220.98" size="1.27" layer="95" xref="yes"/>
@@
 <net name="USART_TX" class="0">
 <segment>
-<pinref part="MODULE5" gate="G$1" pin="UART_TX"/>
+<pinref part="MODULE5" gate="G$1" pin="GND_B"/>
 <wire x1="63.5" y1="218.44" x2="66.04" y2="218.44" width="0.1524" layer="91"/>
 <label x="66.04" y="218.44" size="1.27" layer="95" xref="yes"/>
@@
 <net name="GPIO1" class="0">
 <segment>
-<pinref part="MODULE5" gate="G$1" pin="GPIO1"/>
+<pinref part="MODULE5" gate="G$1" pin="GPIO2"/>
 <wire x1="33.02" y1="220.98" x2="30.48" y2="220.98" width="0.1524" layer="91"/>
 <label x="30.48" y="220.98" size="1.27" layer="95" rot="R180" xref="yes"/>
@@
 <net name="GPIO0" class="0">
 <segment>
-<pinref part="MODULE5" gate="G$1" pin="GPIO0"/>
+<pinref part="MODULE5" gate="G$1" pin="GPIO1"/>
 <wire x1="33.02" y1="223.52" x2="30.48" y2="223.52" width="0.1524" layer="91"/>
 <label x="30.48" y="223.52" size="1.27" layer="95" rot="R180" xref="yes"/>
@@
 <net name="3.3V" class="0">
 <segment>
-<pinref part="MODULE5" gate="G$1" pin="3V3"/>
+<pinref part="MODULE5" gate="G$1" pin="3V3_A"/>
 <wire x1="33.02" y1="233.68" x2="27.94" y2="233.68" width="0.1524" layer="91"/>
 <pinref part="SUPPLY1" gate="G$1" pin="3.3V"/>
@@
 <net name="GND" class="0">
 <segment>
-<pinref part="MODULE5" gate="G$1" pin="GND"/>
+<pinref part="MODULE5" gate="G$1" pin="GND_A"/>
 <pinref part="GND1" gate="G$1" pin="GND"/>
 <wire x1="63.5" y1="233.68" x2="66.04" y2="233.68" width="0.1524" layer="91"/>
